File: CpuSch/RiscV_CPU.sch (KiCad schematic (older format))
At the start: 7 parts

Commit message: Updated main README
Parts:
- U?: value DRam -> DBus
Connections:
- new net: U?.~, U?.~ (OpCode)
- new net: U?.~, U?.~ (PrevPC)
- new net: U?.~, U?.~, U?.~ (PrevPC), U?.~ (RD)
- new net: U?.~, U?.~, U?.~ (PrevPC), U?.~ (WE)
- new net: U?.~, U?.~
- new net: U?.~, U?.~, U?.~ (WE)
- new net: U?.~, U?.~ (WE)
Changed lines of the file:
@@
 EESchema Schematic File Version 4
-LIBS:KiCAD_RiscVCPU-cache
 EELAYER 30 0
 EELAYER END
@@
 P 4225 2500
 F 0 "U?" H 4225 2741 39  0001 C CNN
-F 1 "DRam" H 4225 2666 39  0000 C CNN
+F 1 "DBus" H 4225 2650 39  0000 C CNN
 F 2 "" H 4225 2500 50  0001 C CNN
 F 3 "" H 4225 2500 50  0001 C CNN
